File: garber/cardsize_keyboad.kicad_sch (KiCad schematic)
At the start: 18 parts, among them SW0 Reset_SW, SW1 SW_PUSH, SW2 SW_PUSH, SW3 SW_PUSH, SW4 SW_PUSH, SW5 SW_PUSH, SW6 SW_PUSH, SW7 SW_PUSH, SW8 SW_PUSH, U1 ProMicro

Commit message: FW first commit
Other:
- title: Card size keyboard -> Kuriyokan (Card size keyboard)
Changed lines of the file:
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@@
   (paper "A4")
   (title_block
-    (title "Card size keyboard")
-    (rev "0")
+    (title "Kuriyokan (Card size keyboard)")
+    (rev "1")
     (company "toriten (s51517765)")
   )
